Commit message: feat: 工业机器人真实运动仿真 + G1 步态修复 + 负载颜色映射
工业机器人（交付形态）：
- mock 工业流改为梯形速度插补 + 关节同步运动，4 品牌各自示教程序（FANUC 上下料 / KUKA 装配 / ESTUN 码垛 / YASKAWA 翻腕搬运）
- 运动状态联动：WORKING 跑程序、IDLE 缓慢回 home、ALARM 急停锁定，解除后从当前位置续跑
- 遥测真实化：speed_rpm 由角速度推算、负载/电流随运动强度起伏、温度一阶惯性漂移、TCP 由简化正运动学推导
- 工业数据 2Hz/台广播（原 5s 轮询），告警事件驱动只发一次
- URDF 模型新增关节负载颜色映射：>100% 红 / >80% 黄（自发光）/ 正常恢复品牌原色，材质按 mesh 克隆隔离
- 工业场景差异化：混凝土地面（膨胀缝）+ 螺栓基座（基墩/钢板/地脚螺栓），商用机器人保持原哑光网格地面
- IndustrialRobotModel 关节角 useFrame 插值（τ=0.25s）匹配 2Hz 遥测
- 工业适配器状态直通（idle/error 直传），WS hub 按签名节流工业日志

G1 步态修复（太空步/螃蟹步/转向抽搐）：
- 步频公式改为 速度÷(2×步长)，步幅角按 asin(步长/2/腿长) 物理推导，视觉迈步距离=物理移动距离
- 朝向公式修正为 Ry(-θ)，G1 URDF 前向为局部 +X，旧公式恒侧移 90°（螃蟹步）
- 移除转向位置冻结状态机，改 τ=0.18s 连续航向跟踪 + 速度向量 EMA 滤噪 + 实测 tick 间隔插值
- 抽取 gaitMath.ts 纯函数库（12 个零依赖函数）+ 33 例单元测试（含旧 bug 回归防线）
- digital-twin 接入 vitest 测试基础设施

模型与文档：
- 替换 4 品牌旧 STL 为官方高细节模型（ros-industrial / ESTUN-R-D），URDF 重写真实关节参数
- README 目录树按实际文件修正，FEATURES.md 同步功能清单与变更日志

验证：112 例测试全部通过，tsc 0 错误，浏览器实测断连冻结/恢复续动/负载颜色逐关节精确匹配

File: apps/web-console/public/models/estun/robot.urdf (robot description, URDF)
Before this commit: robot estun_er6, 7 links, 6 joints
Links:
- removed link base
- removed link j1
- removed link j2
- removed link j3
- removed link j4
- removed link j5
- removed link j6
- added link base_link; visual mesh filename=package://estun_support/meshes/base_link.stl
- added link link_1; visual mesh filename=package://estun_support/meshes/link1.stl
- added link link_2; visual mesh filename=package://estun_support/meshes/link2.stl
- added link link_3; visual mesh filename=package://estun_support/meshes/link3.stl
- added link link_4; visual mesh filename=package://estun_support/meshes/link4.stl
- added link link_5; visual mesh filename=package://estun_support/meshes/link5.stl
- added link link_6; visual mesh filename=package://estun_support/meshes/link6.stl
Joints:
- joint joint_1: axis 0 1 0 -> 0 0 -1; child j1 -> link_1; limit lower=-2.967059728 upper=2.967059728 effort=100 velocity=3.14 -> lower=-2.967060 upper=2.967060 effort=500 velocity=5.846853; origin xyz=0 0 0.245 rpy=0 0 0 -> xyz=0 0 0.391 rpy=0 0 0; parent base -> base_link
- joint joint_2: axis 1 0 0 -> 0 1 0; child j2 -> link_2; limit lower=-1.570796327 upper=2.617993878 effort=100 velocity=2.094 -> lower=-1.396263 upper=2.356194 effort=450 velocity=5.759587; origin xyz=0 0 -0.14 rpy=0 0 0 -> xyz=0.040 0 0 rpy=0 0 0; parent j1 -> link_1
- joint joint_3: axis 1 0 0 -> 0 1 0; child j3 -> link_3; limit lower=-2.617993878 upper=1.570796327 effort=100 velocity=2.094 -> lower=-3.316126 upper=1.134464 effort=200 velocity=7.068583; origin xyz=0 0 -0.28 rpy=0 0 0 -> xyz=0 0 0.430 rpy=0 0 0; parent j2 -> link_2
- joint joint_4: axis 1 0 0 -> 0 0 -1; child j4 -> link_4; limit lower=-3.839724354 upper=3.839724354 effort=50 velocity=4.189 -> lower=-3.316126 upper=3.316126 effort=50 velocity=8.726646; origin xyz=0 0 -0.20 rpy=0 0 0 -> xyz=0 0 0.040 rpy=0 1.570796327 0; parent j3 -> link_3
- joint joint_5: child j5 -> link_5; limit lower=-2.443460953 upper=2.443460953 effort=50 velocity=3.141 -> lower=-2.094395 upper=2.094395 effort=50 velocity=7.853982; origin xyz=0 0 -0.09 rpy=0 0 0 -> xyz=0 0 0.445 rpy=0 0 0; parent j4 -> link_4
- joint joint_6: axis 1 0 0 -> 0 0 -1; child j6 -> link_6; limit lower=-6.283185307 upper=6.283185307 effort=30 velocity=6.283 -> lower=-6.283185 upper=6.283185 effort=50 velocity=12.304571; origin xyz=0 0 -0.08 rpy=0 0 0 -> xyz=0 0 0 rpy=0 0 0; parent j5 -> link_5

File: apps/web-console/public/models/fanuc/robot.urdf (robot description, URDF)
Before this commit: robot fanuc_m20id, 7 links, 6 joints
Links:
- removed link base
- removed link j1
- removed link j2
- removed link j3
- removed link j4
- removed link j5
- removed link j6
- added link base_link; visual mesh filename=package://fanuc_support/meshes/base_link.stl
- added link link_1; visual mesh filename=package://fanuc_support/meshes/link_1.stl
- added link link_2; visual mesh filename=package://fanuc_support/meshes/link_2.stl
- added link link_3; visual mesh filename=package://fanuc_support/meshes/link_3.stl
- added link link_4; visual mesh filename=package://fanuc_support/meshes/link_4.stl
- added link link_5; visual mesh filename=package://fanuc_support/meshes/link_5.stl
- added link link_6; visual mesh filename=package://fanuc_support/meshes/link_6.stl
Joints:
- joint joint_1: axis 0 1 0 -> 0 0 1; child j1 -> link_1; limit lower=-2.967059728 upper=2.967059728 effort=100 velocity=3.14 -> lower=-2.967060 upper=2.967060 effort=100 velocity=3.403392; origin xyz=0 0 0.275 rpy=0 0 0 -> xyz=0 0 0.525 rpy=0 0 0; parent base -> base_link
- joint joint_2: axis 1 0 0 -> 0 1 0; child j2 -> link_2; limit lower=-1.570796327 upper=2.617993878 effort=100 velocity=2.094 -> lower=-1.745329 upper=2.792527 effort=100 velocity=3.054326; origin xyz=0 0 -0.15 rpy=0 0 0 -> xyz=0.150 0 0 rpy=0 0 0; parent j1 -> link_1
- joint joint_3: axis 1 0 0 -> 0 -1 0; child j3 -> link_3; limit lower=-2.617993878 upper=1.570796327 effort=100 velocity=2.094 -> lower=-3.228859 upper=4.766843 effort=100 velocity=3.141593; origin xyz=0 0 -0.35 rpy=0 0 0 -> xyz=0 0 0.790 rpy=0 0 0; parent j2 -> link_2
- joint joint_4: axis 1 0 0 -> -1 0 0; child j4 -> link_4; limit lower=-3.839724354 upper=3.839724354 effort=50 velocity=4.189 -> lower=-3.490658 upper=3.490658 effort=50 velocity=6.283185; origin xyz=0 0 -0.25 rpy=0 0 0 -> xyz=0 0 0.250 rpy=0 0 0; parent j3 -> link_3
- joint joint_5: axis 0 1 0 -> 0 -1 0; child j5 -> link_5; limit lower=-2.443460953 upper=2.443460953 effort=50 velocity=3.141 -> lower=-2.443461 upper=2.443461 effort=50 velocity=6.283185; origin xyz=0 0 -0.12 rpy=0 0 0 -> xyz=0.835 0 0 rpy=0 0 0; parent j4 -> link_4
- joint joint_6: axis 1 0 0 -> -1 0 0; child j6 -> link_6; limit lower=-6.283185307 upper=6.283185307 effort=30 velocity=6.283 -> lower=-4.712389 upper=4.712389 effort=30 velocity=9.599311; origin xyz=0 0 -0.10 rpy=0 0 0 -> xyz=0.100 0 0 rpy=0 0 0; parent j5 -> link_5

File: apps/web-console/public/models/kuka/robot.urdf (robot description, URDF)
Before this commit: robot kuka_kr10_r1100, 7 links, 6 joints
Links:
- removed link base
- removed link j1
- removed link j2
- removed link j3
- removed link j4
- removed link j5
- removed link j6
- added link base_link; visual mesh filename=package://kuka_kr10_support/meshes/base_link.stl
- added link link_1; visual mesh filename=package://kuka_kr10_support/meshes/link_1.stl
- added link link_2; visual mesh filename=package://kuka_kr10_support/meshes/link_2.stl
- added link link_3; visual mesh filename=package://kuka_kr10_support/meshes/link_3.stl
- added link link_4; visual mesh filename=package://kuka_kr10_support/meshes/link_4.stl
- added link link_5; visual mesh filename=package://kuka_kr10_support/meshes/link_5.stl
- added link link_6; visual mesh filename=package://kuka_kr10_support/meshes/link_6.stl
Joints:
- removed joint joint_1
- removed joint joint_2
- removed joint joint_3
- removed joint joint_4
- removed joint joint_5
- removed joint joint_6
- added joint joint_a1: type revolute, parent base_link, child link_1, origin xyz=0 0 0.400 rpy=0 0 0, axis 0 0 -1, limit lower=-2.967060 upper=2.967060 effort=100 velocity=6.283185
- added joint joint_a2: type revolute, parent link_1, child link_2, origin xyz=0.025 0 0 rpy=0 0 0, axis 0 1 0, limit lower=-3.316126 upper=0.785398 effort=100 velocity=5.235988
- added joint joint_a3: type revolute, parent link_2, child link_3, origin xyz=0.455 0 0 rpy=0 0 0, axis 0 1 0, limit lower=-2.094395 upper=2.722714 effort=100 velocity=6.283185
- added joint joint_a4: type revolute, parent link_3, child link_4, origin xyz=0 0 0.035 rpy=0 0 0, axis -1 0 0, limit lower=-3.228859 upper=3.228859 effort=50 velocity=6.651684
- added joint joint_a5: type revolute, parent link_4, child link_5, origin xyz=0.420 0 0 rpy=0 0 0, axis 0 1 0, limit lower=-2.094395 upper=2.094395 effort=50 velocity=6.773870
- added joint joint_a6: type revolute, parent link_5, child link_6, origin xyz=0.080 0 0 rpy=0 0 0, axis -1 0 0, limit lower=-6.108652 upper=6.108652 effort=30 velocity=10.733775

File: apps/web-console/public/models/yaskawa/robot.urdf (robot description, URDF)
Before this commit: robot yaskawa_gp7, 7 links, 6 joints
Links:
- removed link base
- removed link j1
- removed link j2
- removed link j3
- removed link j4
- removed link j5
- removed link j6
- added link base_link; visual mesh filename=package://yaskawa_support/meshes/gp7_base_link.stl
- added link link_1_s; visual mesh filename=package://yaskawa_support/meshes/gp7_link_1_s.stl
- added link link_2_l; visual mesh filename=package://yaskawa_support/meshes/gp7_link_2_l.stl
- added link link_3_u; visual mesh filename=package://yaskawa_support/meshes/gp7_link_3_u.stl
- added link link_4_r; visual mesh filename=package://yaskawa_support/meshes/gp7_link_4_r.stl
- added link link_5_b; visual mesh filename=package://yaskawa_support/meshes/gp7_link_5_b.stl
- added link link_6_t; visual mesh filename=package://yaskawa_support/meshes/gp7_link_6_t.stl
Joints:
- removed joint joint_b
- removed joint joint_l
- removed joint joint_r
- removed joint joint_s
- removed joint joint_t
- removed joint joint_u
- added joint joint_1_s: type revolute, parent base_link, child link_1_s, origin xyz=0 0 0.330 rpy=0 0 0, axis 0 0 1, limit lower=-2.967060 upper=2.967060 effort=212.66 velocity=6.544985
- added joint joint_2_l: type revolute, parent link_1_s, child link_2_l, origin xyz=0.040 0 0 rpy=0 0 0, axis 0 1 0, limit lower=-1.134464 upper=2.530727 effort=205.80 velocity=5.497787
- added joint joint_3_u: type revolute, parent link_2_l, child link_3_u, origin xyz=0 0 0.445 rpy=0 0 0, axis 0 -1 0, limit lower=-1.221730 upper=3.316126 effort=106.82 velocity=7.155850
- added joint joint_4_r: type revolute, parent link_3_u, child link_4_r, origin xyz=0.440 0 0.040 rpy=0 0 0, axis -1 0 0, limit lower=-4.712389 upper=4.712389 effort=60.35 velocity=8.726646
- added joint joint_5_b: type revolute, parent link_4_r, child link_5_b, origin xyz=0 0 0 rpy=0 0 0, axis 0 -1 0, limit lower=-2.443461 upper=2.443461 effort=37.13 velocity=8.726646
- added joint joint_6_t: type revolute, parent link_5_b, child link_6_t, origin xyz=0 0 0 rpy=0 0 0, axis -1 0 0, limit lower=-6.283185 upper=6.283185 effort=18.46 velocity=13.962634
